File: synth/MAIN_VFO.sch (KiCad schematic (older format))
At the start: 39 parts

Commit message: automated commit
Parts:
- removed C?: 100nF, symbol Device:CP1
- removed C? (x2): 1uF, symbol Device:CP1
- removed D?: D_Schottky_Small_ALT, symbol Device:D_Schottky_Small_ALT
- removed JP? (x2): SolderJumper_2_Bridged, symbol Jumper:SolderJumper_2_Bridged
- removed Q?: BC549BTA, symbol Device:Q_NPN_CBE
- removed Q?: BC556BTA, symbol Device:Q_PNP_CBE
- removed R?: NP_100, symbol Device:R
- removed R? (x4): 10k, symbol Device:R
- removed R? (x4): 3k3, symbol Device:R
- removed R?: 5k, symbol Device:R
- removed R?: NP_10k, symbol Device:R
- removed RV? (x3): 10k, symbol Device:R_POT
- removed SW?: SW_SPDT, symbol Switch:SW_SPDT
- removed TP? (x10): PTH_1_mm, TestPoint:TestPoint_THTPad_D2.0mm_Drill1.0mm, symbol custom:PTH_1_mm
- removed U?: SE555P, symbol custom:SE555P
- removed U? (x5): MCP6004, Package_DIP:DIP-14_W7.62mm_LongPads, symbol custom:MCP6004
- added C1: 1uF, symbol Device:CP1
- added C2, C3: C, symbol Device:C
- added D1: LED_ALT, symbol Device:LED_ALT
- added JP1: SolderJumper_2_Open, symbol Jumper:SolderJumper_2_Open
- added JP2, JP3, JP4: SolderJumper_2_Bridged, symbol Jumper:SolderJumper_2_Bridged
- added Q1: Q_NMOS_SGD, symbol Device:Q_NMOS_SGD
- added Q2: Q_PMOS_SGD, symbol Device:Q_PMOS_SGD
- added R1, R10, R11, R13, R4: 3k3, symbol Device:R
- added R12: NP_100, symbol Device:R
- added R2: NP, symbol Device:R
- added R3, R5, R6, R7: 10k, symbol Device:R
- added R8, R9: NP_10k, symbol Device:R
- added RV1, RV2, RV3, RV4: 10k, symbol Device:R_POT
- added SW1: SW_SPDT, symbol Switch:SW_SPDT
- added TP1, TP10, TP11, TP12, TP2, TP3, TP4, TP5, TP6, TP7, TP8, TP9: PTH_1_mm, TestPoint:TestPoint_THTPad_D2.0mm_Drill1.0mm, symbol custom:PTH_1_mm
- added U1: MCP6004, Package_DIP:DIP-14_W7.62mm_LongPads, symbol custom:MCP6004
- added U2: SE555P, symbol custom:SE555P
Connections:
- net +5V: now also C1.1, C3.1, JP1.1 (A), R5.2, R7.2, RV3.3, U1.4 (V+), U2.4 (~R), U2.8 (VCC)
- net DISCHARGE: now also D1.1 (K), R4.2, U2.7 (DISCH)
- net GND: now also C1.2, C3.2, R6.1, R9.1, RV3.1, TP11.1, U1.11 (V-), U2.1 (GND)
- net HI_Z_REF: now also U1.3 (+), U1.5 (+)
- net TRIANGLE: now also C2.1, SW1.1 (A), TP8.1, U1.7, U2.2 (TRIG), U2.6 (THR)
- new net: Q1.2 (G), R10.1
- new net: R10.2, R11.2, R3.1, TP12.1, U2.3 (OUT)
- new net: Q2.2 (G), R11.1
- new net: C2.2, JP4.1 (A), R12.2, TP6.1, U1.6 (-)
- new net: JP4.2 (B), R12.1, RV2.2, TP5.1
- new net: R4.1, R5.1, R6.2, R7.1, TP3.1, U1.10 (+)
- new net: JP3.1 (A), R8.2, TP2.1, U1.9 (-)
- new net: JP3.2 (B), R8.1, R9.2, SW1.3 (C), TP4.1, U1.8
- new net: RV3.2, TP9.1, U1.12 (+)
- new net: Q1.3 (D), Q2.3 (D), RV1.2, TP1.1, U1.1
- new net: R13.1, SW1.2 (B), TP7.1
- new net: R13.2, RV4.1, U1.13 (-)
- new net: Q2.1 (S), RV2.1
- new net: Q1.1 (S), RV2.3
- new net: R3.2, RV1.1, U1.2 (-)
- new net: JP1.2 (B), JP2.1 (A), R1.1, R2.1
- new net: D1.2 (A), R1.2, R2.2
- new net VDD_BAT: JP2.2 (B)
- new net VFO_OUT: RV4.2, TP10.1, U1.14
- no-connect marks 2 -> 3
Other:
- note added: "FREQ"
- note removed: "LINEAR"
- note removed: "LOGARITHMIC"

Commit message: automated commit
Parts:
- C1: renamed from C3; footprint (none) -> Capacitor_THT:C_Disc_D3.0mm_W1.6mm_P2.50mm
- C2: footprint (none) -> Capacitor_THT:C_Disc_D3.0mm_W1.6mm_P2.50mm
- C3: renamed from C1; value 1uF -> NP; footprint (none) -> Capacitor_THT:CP_Radial_D6.3mm_P2.50mm; NP NP -> (none)
- D1: footprint (none) -> LED_THT:LED_D5.0mm
- JP1: renamed from JP4; footprint (none) -> Jumper:SolderJumper-2_P1.3mm_Open_RoundedPad1.0x1.5mm
- JP2: renamed from JP1; footprint (none) -> Jumper:SolderJumper-2_P1.3mm_Open_RoundedPad1.0x1.5mm
- JP3: renamed from JP2; footprint (none) -> Jumper:SolderJumper-2_P1.3mm_Open_RoundedPad1.0x1.5mm
- JP4: renamed from JP3; footprint (none) -> Jumper:SolderJumper-2_P1.3mm_Open_RoundedPad1.0x1.5mm
- Q1, Q2: footprint (none) -> Package_TO_SOT_THT:TO-92
- R1: renamed from R3; footprint (none) -> Resistor_THT:R_Axial_DIN0207_L6.3mm_D2.5mm_P10.16mm_Horizontal
- R10: renamed from R1; footprint (none) -> Resistor_THT:R_Axial_DIN0207_L6.3mm_D2.5mm_P10.16mm_Horizontal
- R11: renamed from R2; footprint (none) -> Resistor_THT:R_Axial_DIN0207_L6.3mm_D2.5mm_P10.16mm_Horizontal
- R12: renamed from R8; footprint (none) -> Resistor_THT:R_Axial_DIN0207_L6.3mm_D2.5mm_P10.16mm_Horizontal
- R13: renamed from R9; footprint (none) -> Resistor_THT:R_Axial_DIN0207_L6.3mm_D2.5mm_P10.16mm_Horizontal
- R2: renamed from R10; footprint (none) -> Resistor_THT:R_Axial_DIN0207_L6.3mm_D2.5mm_P10.16mm_Horizontal
- R3: renamed from R12; footprint (none) -> Resistor_THT:R_Axial_DIN0207_L6.3mm_D2.5mm_P10.16mm_Horizontal
- R4: renamed from R11; footprint (none) -> Resistor_THT:R_Axial_DIN0207_L6.3mm_D2.5mm_P10.16mm_Horizontal
- R5: footprint (none) -> Resistor_THT:R_Axial_DIN0207_L6.3mm_D2.5mm_P10.16mm_Horizontal
- R6: renamed from R7; footprint (none) -> Resistor_THT:R_Axial_DIN0207_L6.3mm_D2.5mm_P10.16mm_Horizontal
- R7: renamed from R4; footprint (none) -> Resistor_THT:R_Axial_DIN0207_L6.3mm_D2.5mm_P10.16mm_Horizontal
- R8: renamed from R13; footprint (none) -> Resistor_THT:R_Axial_DIN0207_L6.3mm_D2.5mm_P10.16mm_Horizontal
- R9: renamed from R6; footprint (none) -> Resistor_THT:R_Axial_DIN0207_L6.3mm_D2.5mm_P10.16mm_Horizontal
- RV1, RV2: footprint (none) -> Potentiometer_THT:Potentiometer_Bourns_PTV09A-1_Single_Vertical
- RV3: renamed from RV4; footprint (none) -> Potentiometer_THT:Potentiometer_Bourns_PTV09A-1_Single_Vertical
- RV4: renamed from RV3; footprint (none) -> Potentiometer_THT:Potentiometer_Bourns_PTV09A-1_Single_Vertical
- SW1: footprint (none) -> custom:OS102011MS2QN1
- U1: footprint Package_DIP:DIP-14_W7.62mm_LongPads -> Package_DIP:DIP-14_W7.62mm_Socket
- U2: footprint (none) -> Package_DIP:DIP-8_W7.62mm_Socket
- renumbered TP6 to TP1, TP2 to TP10, TP9 to TP11, TP4 to TP12, TP8 to TP2, TP1 to TP3, TP5 to TP4, TP12 to TP5, TP11 to TP6, TP10 to TP7, TP3 to TP8, TP7 to TP9

Commit message: automated commit
Parts:
- TP1, TP10, TP11, TP12, TP2, TP3, TP4, TP5, TP6, TP7, TP8, TP9: footprint TestPoint:TestPoint_THTPad_D2.0mm_Drill1.0mm -> custom:TestPoint_THTPad_D2.0mm_Drill1.0mm
Changed lines of the file:
@@
 F 0 "TP8" V 5100 4850 50  0000 L BNN
 F 1 "PTH_1_mm" V 5150 4700 50  0001 L BNN
-F 2 "TestPoint:TestPoint_THTPad_D2.0mm_Drill1.0mm" H 4800 4650 50  0001 L BNN
+F 2 "custom:TestPoint_THTPad_D2.0mm_Drill1.0mm" H 4800 4650 50  0001 L BNN
 F 3 "" H 5000 5000 50  0001 L BNN
 	1    5000 4900
@@
 F 0 "TP10" H 4600 5350 50  0000 L BNN
 F 1 "PTH_1_mm" H 4550 5200 50  0001 L BNN
-F 2 "TestPoint:TestPoint_THTPad_D2.0mm_Drill1.0mm" H 4500 5050 50  0001 L BNN
+F 2 "custom:TestPoint_THTPad_D2.0mm_Drill1.0mm" H 4500 5050 50  0001 L BNN
 F 3 "" H 4700 5400 50  0001 L BNN
 	1    4700 5300
@@
 F 0 "TP12" H 6200 5850 50  0000 L BNN
 F 1 "PTH_1_mm" H 6150 5700 50  0001 L BNN
-F 2 "TestPoint:TestPoint_THTPad_D2.0mm_Drill1.0mm" H 6100 5550 50  0001 L BNN
+F 2 "custom:TestPoint_THTPad_D2.0mm_Drill1.0mm" H 6100 5550 50  0001 L BNN
 F 3 "" H 6300 5900 50  0001 L BNN
 	1    6300 5800
@@
 F 0 "TP7" V 9100 4550 50  0000 L BNN
 F 1 "PTH_1_mm" V 9150 4400 50  0001 L BNN
-F 2 "TestPoint:TestPoint_THTPad_D2.0mm_Drill1.0mm" H 8800 4350 50  0001 L BNN
+F 2 "custom:TestPoint_THTPad_D2.0mm_Drill1.0mm" H 8800 4350 50  0001 L BNN
 F 3 "" H 9000 4700 50  0001 L BNN
 	1    9000 4600
@@
 F 0 "TP11" H 8450 5750 50  0000 L BNN
 F 1 "PTH_1_mm" H 8250 5650 50  0001 L BNN
-F 2 "TestPoint:TestPoint_THTPad_D2.0mm_Drill1.0mm" H 8200 5500 50  0001 L BNN
+F 2 "custom:TestPoint_THTPad_D2.0mm_Drill1.0mm" H 8200 5500 50  0001 L BNN
 F 3 "" H 8400 5850 50  0001 L BNN
 	1    8400 5750
@@
 F 0 "TP3" V 4800 1650 50  0000 L BNN
 F 1 "PTH_1_mm" V 4850 1500 50  0001 L BNN
-F 2 "TestPoint:TestPoint_THTPad_D2.0mm_Drill1.0mm" H 4500 1450 50  0001 L BNN
+F 2 "custom:TestPoint_THTPad_D2.0mm_Drill1.0mm" H 4500 1450 50  0001 L BNN
 F 3 "" H 4700 1800 50  0001 L BNN
 	1    4700 1700
@@
 F 0 "TP4" V 6450 1650 50  0000 L BNN
 F 1 "PTH_1_mm" V 6500 1500 50  0001 L BNN
-F 2 "TestPoint:TestPoint_THTPad_D2.0mm_Drill1.0mm" H 6150 1450 50  0001 L BNN
+F 2 "custom:TestPoint_THTPad_D2.0mm_Drill1.0mm" H 6150 1450 50  0001 L BNN
 F 3 "" H 6350 1800 50  0001 L BNN
 	1    6350 1700
@@
 F 0 "TP1" V 7200 1550 50  0000 L BNN
 F 1 "PTH_1_mm" V 7250 1400 50  0001 L BNN
-F 2 "TestPoint:TestPoint_THTPad_D2.0mm_Drill1.0mm" H 6900 1350 50  0001 L BNN
+F 2 "custom:TestPoint_THTPad_D2.0mm_Drill1.0mm" H 6900 1350 50  0001 L BNN
 F 3 "" H 7100 1700 50  0001 L BNN
 	1    7100 1600
@@
 F 0 "TP6" H 9700 2800 50  0000 L BNN
 F 1 "PTH_1_mm" H 9650 2650 50  0001 L BNN
-F 2 "TestPoint:TestPoint_THTPad_D2.0mm_Drill1.0mm" H 9600 2500 50  0001 L BNN
+F 2 "custom:TestPoint_THTPad_D2.0mm_Drill1.0mm" H 9600 2500 50  0001 L BNN
 F 3 "" H 9800 2850 50  0001 L BNN
 	1    9800 2750
@@
 F 0 "TP2" V 8100 1550 50  0000 L BNN
 F 1 "PTH_1_mm" V 8150 1400 50  0001 L BNN
-F 2 "TestPoint:TestPoint_THTPad_D2.0mm_Drill1.0mm" H 7800 1350 50  0001 L BNN
+F 2 "custom:TestPoint_THTPad_D2.0mm_Drill1.0mm" H 7800 1350 50  0001 L BNN
 F 3 "" H 8000 1700 50  0001 L BNN
 	1    8000 1600
@@
 F 0 "TP5" V 10050 1900 50  0000 L BNN
 F 1 "PTH_1_mm" V 10100 1750 50  0001 L BNN
-F 2 "TestPoint:TestPoint_THTPad_D2.0mm_Drill1.0mm" H 9750 1700 50  0001 L BNN
+F 2 "custom:TestPoint_THTPad_D2.0mm_Drill1.0mm" H 9750 1700 50  0001 L BNN
 F 3 "" H 9950 2050 50  0001 L BNN
 	1    9950 1950
@@
 F 0 "TP9" V 7550 4850 50  0000 L BNN
 F 1 "PTH_1_mm" V 7600 4700 50  0001 L BNN
-F 2 "TestPoint:TestPoint_THTPad_D2.0mm_Drill1.0mm" H 7250 4650 50  0001 L BNN
+F 2 "custom:TestPoint_THTPad_D2.0mm_Drill1.0mm" H 7250 4650 50  0001 L BNN
 F 3 "" H 7450 5000 50  0001 L BNN
 	1    7450 4900
