File: synth/MAIN_VFO.sch (KiCad schematic (older format))
At the start: 41 parts, among them Q1 Q_NMOS_SGD, Q2 Q_PMOS_SGD, SW1 SW_SPDT, U1 MCP6004, U2 SE555P

Commit message: automated commit
Parts:
- D1: value LED_ALT -> LED
- JP1, JP2: renamed from JP?; value SolderJumper_2_Bridged -> SolderJumper_Bridged
- JP3: renamed from JP?; value SolderJumper_2_Open -> SolderJumper_Open; footprint (none) -> Jumper:SolderJumper-2_P1.3mm_Open_RoundedPad1.0x1.5mm
- R10, R12: renamed from R?; value 1k0 -> 1k
- R11: value 1k0 -> 1k
- R3: value NP -> NP_100
- RV5: renamed from RV?; value 1k0 -> 1k; footprint Potentiometer_THT:Potentiometer_Bourns_PTV09A-1_Single_Vertical -> custom:CT6EP102
- gave numbers to parts that had none: 2
Changed lines of the file:
@@
 AR Path="/5E826FFF/5E78F71D" Ref="R?"  Part="1"
 F 0 "R3" V 6675 2250 50  0000 L CNN
-F 1 "NP" V 6600 2250 39  0000 C CNN
+F 1 "NP_100" V 6600 2250 31  0000 C CNN
 F 2 "Resistor_THT:R_Axial_DIN0207_L6.3mm_D2.5mm_P10.16mm_Horizontal" V 6530 2250 50  0001 C CNN
 F 3 "~" H 6600 2250 50  0001 C CNN
@@
 P 1800 6850
 F 0 "D1" H 1800 6950 50  0000 C CNN
-F 1 "LED_ALT" H 1800 6750 50  0001 C CNN
+F 1 "LED" H 1800 6750 50  0001 C CNN
 F 2 "LED_THT:LED_D5.0mm" H 1800 6850 50  0001 C CNN
 F 3 "~" H 1800 6850 50  0001 C CNN
@@
 AR Path="/5E826FFF/5E8E14D7" Ref="R?"  Part="1"
 F 0 "R11" V 1700 6250 50  0000 L CNN
-F 1 "1k0" V 1800 6300 39  0000 L CNN
+F 1 "1k" V 1800 6300 39  0000 L CNN
 F 2 "Resistor_THT:R_Axial_DIN0207_L6.3mm_D2.5mm_P10.16mm_Horizontal" V 1730 6350 50  0001 C CNN
 F 3 "~" H 1800 6350 50  0001 C CNN
@@
 P 6600 1900
 AR Path="/5E4A00FF/5EB0ACDA" Ref="JP?"  Part="1"
-AR Path="/5E4A013A/5EB0ACDA" Ref="JP?"  Part="1"
+AR Path="/5E4A013A/5EB0ACDA" Ref="JP1"  Part="1"
 AR Path="/5E826FFF/5EB0ACDA" Ref="JP?"  Part="1"
-F 0 "JP?" H 6600 1800 50  0000 C CNN
-F 1 "SolderJumper_2_Bridged" H 6600 1800 50  0001 C CNN
+F 0 "JP1" H 6600 1800 50  0000 C CNN
+F 1 "SolderJumper_Bridged" H 6600 1800 50  0001 C CNN
 F 2 "Jumper:SolderJumper-2_P1.3mm_Open_RoundedPad1.0x1.5mm" H 6600 1900 50  0001 C CNN
 F 3 "~" H 6600 1900 50  0001 C CNN
@@
 P 1550 4350
 AR Path="/5E4A00FF/5EB370FB" Ref="RV?"  Part="1"
-AR Path="/5E4A013A/5EB370FB" Ref="RV?"  Part="1"
+AR Path="/5E4A013A/5EB370FB" Ref="RV5"  Part="1"
 AR Path="/5E826FFF/5EB370FB" Ref="RV?"  Part="1"
-F 0 "RV?" V 1450 4450 50  0000 R CNN
-F 1 "1k0" V 1550 4400 39  0000 R CNN
-F 2 "Potentiometer_THT:Potentiometer_Bourns_PTV09A-1_Single_Vertical" H 1550 4350 50  0001 C CNN
+F 0 "RV5" V 1450 4450 50  0000 R CNN
+F 1 "1k" V 1550 4400 39  0000 R CNN
+F 2 "custom:CT6EP102" H 1550 4350 50  0001 C CNN
 F 3 "~" H 1550 4350 50  0001 C CNN
 	1    1550 4350
@@
 P 1550 3950
 AR Path="/5E4A00FF/5EB373D2" Ref="R?"  Part="1"
-AR Path="/5E4A013A/5EB373D2" Ref="R?"  Part="1"
+AR Path="/5E4A013A/5EB373D2" Ref="R10"  Part="1"
 AR Path="/5E826FFF/5EB373D2" Ref="R?"  Part="1"
-F 0 "R?" V 1450 3850 50  0000 L CNN
-F 1 "1k0" V 1550 3900 39  0000 L CNN
+F 0 "R10" V 1450 3850 50  0000 L CNN
+F 1 "1k" V 1550 3900 39  0000 L CNN
 F 2 "Resistor_THT:R_Axial_DIN0207_L6.3mm_D2.5mm_P10.16mm_Horizontal" V 1480 3950 50  0001 C CNN
 F 3 "~" H 1550 3950 50  0001 C CNN
@@
 P 1550 4750
 AR Path="/5E4A00FF/5EB390AA" Ref="R?"  Part="1"
-AR Path="/5E4A013A/5EB390AA" Ref="R?"  Part="1"
+AR Path="/5E4A013A/5EB390AA" Ref="R12"  Part="1"
 AR Path="/5E826FFF/5EB390AA" Ref="R?"  Part="1"
-F 0 "R?" V 1450 4650 50  0000 L CNN
-F 1 "1k0" V 1550 4700 39  0000 L CNN
+F 0 "R12" V 1450 4650 50  0000 L CNN
+F 1 "1k" V 1550 4700 39  0000 L CNN
 F 2 "Resistor_THT:R_Axial_DIN0207_L6.3mm_D2.5mm_P10.16mm_Horizontal" V 1480 4750 50  0001 C CNN
 F 3 "~" H 1550 4750 50  0001 C CNN
@@
 P 1550 3700
 AR Path="/5E4A00FF/5EB43153" Ref="#PWR?"  Part="1"
-AR Path="/5E4A013A/5EB43153" Ref="#PWR?"  Part="1"
+AR Path="/5E4A013A/5EB43153" Ref="#PWR012"  Part="1"
 AR Path="/5E826FFF/5EB43153" Ref="#PWR?"  Part="1"
-F 0 "#PWR?" H 1550 3550 50  0001 C CNN
+F 0 "#PWR012" H 1550 3550 50  0001 C CNN
 F 1 "+5V" H 1550 3840 50  0000 C CNN
 F 2 "" H 1550 3700 50  0001 C CNN
@@
 AR Path="/5E4A00E6/5EB4443C" Ref="#PWR?"  Part="1"
 AR Path="/5E4A00FF/5EB4443C" Ref="#PWR?"  Part="1"
-AR Path="/5E4A013A/5EB4443C" Ref="#PWR?"  Part="1"
+AR Path="/5E4A013A/5EB4443C" Ref="#PWR016"  Part="1"
 AR Path="/5E826FFF/5EB4443C" Ref="#PWR?"  Part="1"
-F 0 "#PWR?" H 1750 4850 50  0001 C CNN
+F 0 "#PWR016" H 1750 4850 50  0001 C CNN
 F 1 "GND" H 1755 4927 50  0000 C CNN
 F 2 "" H 1750 5100 50  0001 C CNN
@@
 P 7050 2450
 AR Path="/5E4A00FF/5EB9836F" Ref="JP?"  Part="1"
-AR Path="/5E4A013A/5EB9836F" Ref="JP?"  Part="1"
+AR Path="/5E4A013A/5EB9836F" Ref="JP2"  Part="1"
 AR Path="/5E826FFF/5EB9836F" Ref="JP?"  Part="1"
-F 0 "JP?" H 7050 2350 50  0000 C CNN
-F 1 "SolderJumper_2_Bridged" H 7050 2350 50  0001 C CNN
+F 0 "JP2" H 7050 2350 50  0000 C CNN
+F 1 "SolderJumper_Bridged" H 7050 2350 50  0001 C CNN
 F 2 "Jumper:SolderJumper-2_P1.3mm_Open_RoundedPad1.0x1.5mm" H 7050 2450 50  0001 C CNN
 F 3 "~" H 7050 2450 50  0001 C CNN
@@
 	6500 2450 6900 2450
 $Comp
-L Jumper:SolderJumper_2_Open JP?
+L Jumper:SolderJumper_2_Open JP3
 U 1 1 5EBA5A64
 P 7050 2700
-F 0 "JP?" H 7050 2780 50  0000 C CNN
-F 1 "SolderJumper_2_Open" H 7050 2600 50  0001 C CNN
-F 2 "" H 7050 2700 50  0001 C CNN
+F 0 "JP3" H 7050 2780 50  0000 C CNN
+F 1 "SolderJumper_Open" H 7050 2600 50  0001 C CNN
+F 2 "Jumper:SolderJumper-2_P1.3mm_Open_RoundedPad1.0x1.5mm" H 7050 2700 50  0001 C CNN
 F 3 "~" H 7050 2700 50  0001 C CNN
 	1    7050 2700
@@
 	1950 4350 2250 4350
 $Comp
-L Device:C C?
+L Device:C C4
 U 1 1 5EC07744
 P 1950 4700
-AR Path="/5E4A013A/5EC07744" Ref="C?"  Part="1"
+AR Path="/5E4A013A/5EC07744" Ref="C4"  Part="1"
 AR Path="/5E826FFF/5EC07744" Ref="C?"  Part="1"
-F 0 "C?" H 1975 4800 50  0000 L CNN
+F 0 "C4" H 1975 4800 50  0000 L CNN
 F 1 "10nF" H 1975 4600 50  0000 L CNN
 F 2 "Capacitor_THT:C_Disc_D3.0mm_W1.6mm_P2.50mm" H 1988 4550 50  0001 C CNN
@@
 $EndComp
 $Comp
-L Device:C C?
+L Device:C C3
 U 1 1 5EC07BEE
 P 1300 2250
-AR Path="/5E4A013A/5EC07BEE" Ref="C?"  Part="1"
+AR Path="/5E4A013A/5EC07BEE" Ref="C3"  Part="1"
 AR Path="/5E826FFF/5EC07BEE" Ref="C?"  Part="1"
-F 0 "C?" H 1325 2350 50  0000 L CNN
+F 0 "C3" H 1325 2350 50  0000 L CNN
 F 1 "10nF" H 1325 2150 50  0000 L CNN
 F 2 "Capacitor_THT:C_Disc_D3.0mm_W1.6mm_P2.50mm" H 1338 2100 50  0001 C CNN

Commit message: automated commit
Parts:
- added JP4, JP5, JP7: SolderJumper_Open, Jumper:SolderJumper-2_P1.3mm_Open_RoundedPad1.0x1.5mm, symbol Jumper:SolderJumper_2_Open
- added R13, R16, R17: 1k, Resistor_THT:R_Axial_DIN0207_L6.3mm_D2.5mm_P10.16mm_Horizontal, symbol Device:R
Connections:
- net at RV2.1: now also JP5.2 (B), R16.2; no longer Q1.1 (S)
- net at RV2.3: now also JP7.1 (A), R17.1; no longer Q2.1 (S)
- net at R1.2, U1.2 (-): now also JP4.2 (B), R13.2; no longer RV1.3
- new net: JP4.1 (A), R13.1, RV1.3
- new net: JP5.1 (A), Q1.1 (S), R16.1
- new net: JP7.2 (B), Q2.1 (S), R17.2
Other:
- moved on the sheet: Q1, Q2, R4, RV1, TP3
Changed lines of the file:
@@
 L Device:R R?
 U 1 1 5E78F562
-P 5500 2700
+P 5500 3100
 AR Path="/5E4A00FF/5E78F562" Ref="R?"  Part="1"
 AR Path="/5E4A013A/5E78F562" Ref="R4"  Part="1"
 AR Path="/5E826FFF/5E78F562" Ref="R?"  Part="1"
-F 0 "R4" V 5600 2600 50  0000 L CNN
-F 1 "3k3" V 5500 2650 39  0000 L CNN
-F 2 "Resistor_THT:R_Axial_DIN0207_L6.3mm_D2.5mm_P10.16mm_Horizontal" V 5430 2700 50  0001 C CNN
-F 3 "~" H 5500 2700 50  0001 C CNN
-	1    5500 2700
+F 0 "R4" V 5600 3000 50  0000 L CNN
+F 1 "3k3" V 5500 3050 39  0000 L CNN
+F 2 "Resistor_THT:R_Axial_DIN0207_L6.3mm_D2.5mm_P10.16mm_Horizontal" V 5430 3100 50  0001 C CNN
+F 3 "~" H 5500 3100 50  0001 C CNN
+	1    5500 3100
 	0    1    -1   0
 $EndComp
@@
 L custom:PTH_1_mm TP?
 U 1 1 5E78F601
-P 4700 1700
+P 4700 1075
 AR Path="/5E4A00FF/5E78F601" Ref="TP?"  Part="1"
 AR Path="/5E4A013A/5E78F601" Ref="TP3"  Part="1"
 AR Path="/5E826FFF/5E78F601" Ref="TP?"  Part="1"
-F 0 "TP3" V 4800 1650 50  0000 L BNN
-F 1 "PTH_1_mm" V 4850 1500 50  0001 L BNN
-F 2 "custom:TestPoint_THTPad_D2.0mm_Drill1.0mm" H 4500 1450 50  0001 L BNN
-F 3 "" H 4700 1800 50  0001 L BNN
-	1    4700 1700
+F 0 "TP3" V 4800 1025 50  0000 L BNN
+F 1 "PTH_1_mm" V 4850 875 50  0001 L BNN
+F 2 "custom:TestPoint_THTPad_D2.0mm_Drill1.0mm" H 4500 825 50  0001 L BNN
+F 3 "" H 4700 1175 50  0001 L BNN
+	1    4700 1075
 	0    -1   -1   0
 $EndComp
@@
 $EndComp
 Wire Wire Line
-	3250 3350 3250 2700
-Wire Wire Line
-	9950 3350 3250 3350
-Wire Wire Line
-	3800 2050 3800 2200
+	3250 3625 3250 3100
+Wire Wire Line
+	9950 3625 3250 3625
+Wire Wire Line
+	3800 1925 3800 2000
 Wire Wire Line
 	4000 2200 3800 2200
@@
 VFO_OUT
 Wire Wire Line
-	5250 2700 5350 2700
-Wire Wire Line
-	5650 2700 5700 2700
+	5250 3100 5350 3100
+Wire Wire Line
+	5650 3100 5700 3100
 Text Notes 8000 4500 0    79   ~ 16
 AMP
 Wire Wire Line
 	3250 2200 3350 2200
-Connection ~ 5250 2700
-Wire Wire Line
-	3250 2700 5250 2700
-Connection ~ 3250 2700
-Wire Wire Line
-	3250 2700 3250 2200
+Connection ~ 5250 3100
+Wire Wire Line
+	3250 3100 5250 3100
 $Comp
 L Device:R R?
@@
 Text Notes 5800 2300 2    79   ~ 16
 DUTY
-Text Notes 3650 1600 0    79   ~ 16
+Text Notes 3650 1075 0    79   ~ 16
 FREQ
 Wire Wire Line
@@
 $EndComp
 Wire Wire Line
-	6000 2900 6000 3000
-Wire Wire Line
-	6000 1500 6000 1600
+	6000 3300 6000 3400
+Wire Wire Line
+	6000 1075 6000 1175
 $Comp
 L Device:R_POT RV?
@@
 $EndComp
 Wire Wire Line
-	4700 1850 4700 1900
-Wire Wire Line
-	4700 1900 4700 2300
-Connection ~ 4700 1900
-Wire Wire Line
-	3950 1900 4700 1900
+	4700 1300 4700 2300
+Connection ~ 4700 1300
+Wire Wire Line
+	3950 1300 4700 1300
 Wire Wire Line
 	8600 1850 8600 2150
 Wire Wire Line
 	9600 1850 9600 2350
-NoConn ~ 3800 1700
-Wire Wire Line
-	3800 1750 3800 1700
+NoConn ~ 3800 1100
+Wire Wire Line
+	3800 1150 3800 1100
 $Comp
 L Device:R_POT RV?
 U 1 1 5E78F70A
-P 3800 1900
+P 3800 1300
 AR Path="/5E4A00FF/5E78F70A" Ref="RV?"  Part="1"
 AR Path="/5E4A013A/5E78F70A" Ref="RV1"  Part="1"
 AR Path="/5E826FFF/5E78F70A" Ref="RV?"  Part="1"
-F 0 "RV1" V 3700 2000 50  0000 R CNN
-F 1 "10k" V 3800 1950 39  0000 R CNN
-F 2 "Potentiometer_THT:Potentiometer_Bourns_PTV09A-1_Single_Vertical" H 3800 1900 50  0001 C CNN
-F 3 "~" H 3800 1900 50  0001 C CNN
-	1    3800 1900
+F 0 "RV1" V 3700 1400 50  0000 R CNN
+F 1 "10k" V 3800 1350 39  0000 R CNN
+F 2 "Potentiometer_THT:Potentiometer_Bourns_PTV09A-1_Single_Vertical" H 3800 1300 50  0001 C CNN
+F 3 "~" H 3800 1300 50  0001 C CNN
+	1    3800 1300
 	1    0    0    -1
 $EndComp
@@
 L Device:Q_NMOS_SGD Q1
 U 1 1 5E7C5A19
-P 5900 1800
+P 5900 1375
 AR Path="/5E4A013A/5E7C5A19" Ref="Q1"  Part="1"
 AR Path="/5E826FFF/5E7C5A19" Ref="Q?"  Part="1"
-F 0 "Q1" H 6100 1850 50  0000 L CNN
-F 1 "Q_NMOS_SGD" H 6100 1750 50  0001 L CNN
-F 2 "Package_TO_SOT_THT:TO-92" H 6100 1900 50  0001 C CNN
-F 3 "~" H 5900 1800 50  0001 C CNN
-	1    5900 1800
+F 0 "Q1" H 6100 1425 50  0000 L CNN
+F 1 "Q_NMOS_SGD" H 6100 1325 50  0001 L CNN
+F 2 "Package_TO_SOT_THT:TO-92" H 6100 1475 50  0001 C CNN
+F 3 "~" H 5900 1375 50  0001 C CNN
+	1    5900 1375
 	1    0    0    -1
 $EndComp
@@
 L Device:Q_PMOS_SGD Q2
 U 1 1 5E9B1FC7
-P 5900 2700
+P 5900 3100
 AR Path="/5E4A013A/5E9B1FC7" Ref="Q2"  Part="1"
 AR Path="/5E826FFF/5E9B1FC7" Ref="Q?"  Part="1"
-F 0 "Q2" H 6100 2750 50  0000 L CNN
-F 1 "Q_PMOS_SGD" H 6100 2650 50  0001 L CNN
-F 2 "Package_TO_SOT_THT:TO-92" H 6100 2800 50  0001 C CNN
-F 3 "~" H 5900 2700 50  0001 C CNN
-	1    5900 2700
+F 0 "Q2" H 6100 3150 50  0000 L CNN
+F 1 "Q_PMOS_SGD" H 6100 3050 50  0001 L CNN
+F 2 "Package_TO_SOT_THT:TO-92" H 6100 3200 50  0001 C CNN
+F 3 "~" H 5900 3100 50  0001 C CNN
+	1    5900 3100
 	1    0    0    1
 $EndComp
@@
 $EndComp
 Wire Wire Line
-	9950 2150 9950 3350
+	9950 2150 9950 3625
 Text Label 2300 7300 2    50   ~ 0
 DISCHARGE
@@
 $EndComp
 Wire Wire Line
-	4600 2300 4700 2300
-Wire Wire Line
 	1800 7000 1800 7300
 Wire Wire Line
@@
 $EndComp
 Wire Wire Line
-	5250 2400 5250 2700
-Wire Wire Line
-	5250 1800 5700 1800
-Wire Wire Line
-	5250 1800 5250 2100
-Wire Wire Line
-	6000 3000 5050 3000
-Wire Wire Line
-	5050 1500 6000 1500
-Connection ~ 4700 2300
-Wire Wire Line
-	4700 2300 5050 2300
-Wire Wire Line
-	5050 2300 5050 3000
-Connection ~ 5050 2300
-Wire Wire Line
-	5050 1500 5050 2300
-Wire Wire Line
-	6000 2400 6000 2500
-Wire Wire Line
-	6000 2000 6000 2100
+	5250 1375 5700 1375
+Wire Wire Line
+	6000 3400 5050 3400
+Wire Wire Line
+	5050 1075 6000 1075
 Wire Wire Line
 	6150 2250 6350 2250
@@
 	5150 5300 5150 5600
 Connection ~ 6100 5600
+$Comp
+L Device:R R?
+U 1 1 5F17FC5A
+P 3800 1775
+AR Path="/5E4A00FF/5F17FC5A" Ref="R?"  Part="1"
+AR Path="/5E4A013A/5F17FC5A" Ref="R13"  Part="1"
+AR Path="/5E826FFF/5F17FC5A" Ref="R?"  Part="1"
+F 0 "R13" V 3700 1675 50  0000 L CNN
+F 1 "1k" V 3800 1725 39  0000 L CNN
+F 2 "Resistor_THT:R_Axial_DIN0207_L6.3mm_D2.5mm_P10.16mm_Horizontal" V 3730 1775 50  0001 C CNN
+F 3 "~" H 3800 1775 50  0001 C CNN
+	1    3800 1775
+	-1   0    0    -1
+$EndComp
+Wire Wire Line
+	4600 2300 4700 2300
+Connection ~ 4700 2300
+Wire Wire Line
+	4700 2300 5050 2300
+Wire Wire Line
+	3800 1625 3800 1575
+Wire Wire Line
+	4700 1225 4700 1300
+$Comp
+L Jumper:SolderJumper_2_Open JP4
+U 1 1 5F1B88E7
+P 3650 1775
+F 0 "JP4" H 3650 1855 50  0000 C CNN
+F 1 "SolderJumper_Open" H 3650 1675 50  0001 C CNN
+F 2 "Jumper:SolderJumper-2_P1.3mm_Open_RoundedPad1.0x1.5mm" H 3650 1775 50  0001 C CNN
+F 3 "~" H 3650 1775 50  0001 C CNN
+	1    3650 1775
+	0    -1   1    0
+$EndComp
+Wire Wire Line
+	3650 1925 3650 2000
+Wire Wire Line
+	3650 2000 3800 2000
+Connection ~ 3800 2000
+Wire Wire Line
+	3800 2000 3800 2200
+Wire Wire Line
+	3650 1625 3650 1575
+Wire Wire Line
+	3650 1575 3800 1575
+Connection ~ 3800 1575
+Wire Wire Line
+	3800 1575 3800 1450
+Wire Wire Line
+	5050 2300 5050 3400
+Wire Wire Line
+	5250 2400 5250 3100
+Wire Wire Line
+	5050 1075 5050 2300
+Wire Wire Line
+	5250 1375 5250 2100
+Wire Wire Line
+	6000 1975 6000 2050
+$Comp
+L Device:R R?
+U 1 1 5F21ADE3
+P 6000 1825
+AR Path="/5E4A00FF/5F21ADE3" Ref="R?"  Part="1"
+AR Path="/5E4A013A/5F21ADE3" Ref="R16"  Part="1"
+AR Path="/5E826FFF/5F21ADE3" Ref="R?"  Part="1"
+F 0 "R16" V 5900 1725 50  0000 L CNN
+F 1 "1k" V 6000 1775 39  0000 L CNN
+F 2 "Resistor_THT:R_Axial_DIN0207_L6.3mm_D2.5mm_P10.16mm_Horizontal" V 5930 1825 50  0001 C CNN
+F 3 "~" H 6000 1825 50  0001 C CNN
+	1    6000 1825
+	-1   0    0    -1
+$EndComp
+Wire Wire Line
+	6000 1675 6000 1625
+$Comp
+L Jumper:SolderJumper_2_Open JP5
+U 1 1 5F21ADEB
+P 5850 1825
+F 0 "JP5" H 5850 1905 50  0000 C CNN
+F 1 "SolderJumper_Open" H 5850 1725 50  0001 C CNN
+F 2 "Jumper:SolderJumper-2_P1.3mm_Open_RoundedPad1.0x1.5mm" H 5850 1825 50  0001 C CNN
+F 3 "~" H 5850 1825 50  0001 C CNN
+	1    5850 1825
+	0    -1   1    0
+$EndComp
+Wire Wire Line
+	5850 1975 5850 2050
+Wire Wire Line
+	5850 1675 5850 1625
+Connection ~ 3250 3100
+Wire Wire Line
+	3250 2200 3250 3100
+Connection ~ 5050 2300
+$Comp
+L Device:R R?
+U 1 1 5F231B39
+P 6000 2650
+AR Path="/5E4A00FF/5F231B39" Ref="R?"  Part="1"
+AR Path="/5E4A013A/5F231B39" Ref="R17"  Part="1"
+AR Path="/5E826FFF/5F231B39" Ref="R?"  Part="1"
+F 0 "R17" V 5900 2550 50  0000 L CNN
+F 1 "1k" V 6000 2600 39  0000 L CNN
+F 2 "Resistor_THT:R_Axial_DIN0207_L6.3mm_D2.5mm_P10.16mm_Horizontal" V 5930 2650 50  0001 C CNN
+F 3 "~" H 6000 2650 50  0001 C CNN
+	1    6000 2650
+	-1   0    0    -1
+$EndComp
+$Comp
+L Jumper:SolderJumper_2_Open JP7
+U 1 1 5F231B41
+P 5850 2650
+F 0 "JP7" H 5850 2730 50  0000 C CNN
+F 1 "SolderJumper_Open" H 5850 2550 50  0001 C CNN
+F 2 "Jumper:SolderJumper-2_P1.3mm_Open_RoundedPad1.0x1.5mm" H 5850 2650 50  0001 C CNN
+F 3 "~" H 5850 2650 50  0001 C CNN
+	1    5850 2650
+	0    -1   1    0
+$EndComp
+Wire Wire Line
+	5850 2800 5850 2875
+Wire Wire Line
+	5850 2500 5850 2450
+Wire Wire Line
+	6000 2400 6000 2450
+Wire Wire Line
+	6000 2800 6000 2875
+Wire Wire Line
+	6000 2875 5850 2875
+Connection ~ 6000 2875
+Wire Wire Line
+	6000 2875 6000 2900
+Wire Wire Line
+	5850 2450 6000 2450
+Connection ~ 6000 2450
+Wire Wire Line
+	6000 2450 6000 2500
+Wire Wire Line
+	5850 2050 6000 2050
+Wire Wire Line
+	6000 2100 6000 2050
+Connection ~ 6000 2050
+Wire Wire Line
+	5850 1625 6000 1625
+Wire Wire Line
+	6000 1575 6000 1625
+Connection ~ 6000 1625
 $EndSCHEMATC

Commit message: automated commit
Parts:
- removed JP1, JP2: SolderJumper_Bridged, Jumper:SolderJumper-2_P1.3mm_Open_RoundedPad1.0x1.5mm, symbol Jumper:SolderJumper_2_Bridged
- removed JP3, JP7: SolderJumper_Open, Jumper:SolderJumper-2_P1.3mm_Open_RoundedPad1.0x1.5mm, symbol Jumper:SolderJumper_2_Open
- removed Q1: Q_NMOS_SGD, Package_TO_SOT_THT:TO-92, symbol Device:Q_NMOS_SGD
- removed Q2: Q_PMOS_SGD, Package_TO_SOT_THT:TO-92, symbol Device:Q_PMOS_SGD
- removed R16, R17: 1k, Resistor_THT:R_Axial_DIN0207_L6.3mm_D2.5mm_P10.16mm_Horizontal, symbol Device:R
- added Q1: 2N3904, Package_TO_SOT_THT:TO-92_Inline, symbol Transistor_BJT:2N3904
- added Q2: 2N3906, Package_TO_SOT_THT:TO-92_Inline, symbol Transistor_BJT:2N3906
- C2: value 10nF -> 100nF
- R10, R11, R12, R13, RV5: value 1k -> 1k0
- R3: value NP_100 -> 1k0
- renumbered JP5 to JP1, JP4 to JP2
Connections:
- net TRIM: now also U1.5 (+)
- net at R2.1: now also Q1.2 (B)
- net at R4.1: now also Q2.2 (B)
- net at RV1.2, TP3.1, U1.1: now also Q1.1 (E), Q2.1 (E)
- net at RV2.2, TP4.1: now also JP1.2 (B), R3.2; no longer R3.1
- net at C2.2, TP1.1, U1.6 (-): now also JP1.1 (A), R3.1; no longer R3.2
- net at RV2.1: now also Q1.3 (C); no longer JP1.2 (B)
- net at RV2.3: now also Q2.3 (C)
Other:
- moved on the sheet: JP1, R4
