File: synth/OUTPUT.sch (KiCad schematic (older format))
At the start: 16 parts, among them J2 Screw_Terminal_01x02, Q3 NP, Q4 NP, SW3 SW_SPDT, U4 MCP6002

Commit message: automated commit
Parts:
- J2: footprint custom:TERMINAL_BLOCK_1x2 -> TerminalBlock:TerminalBlock_bornier-2_P5.08mm
- JP6: value SolderJumper_2_Bridged -> SolderJumper_Bridged
- Q3: value NP -> NP_NPN_CBE
- Q4: value NP -> NP_PNP_CBE
- R19, R23: value NP_10k -> NP_47
- R20, R24, R25: value NP_10k -> NP_3k3
- gave numbers to parts that had none: 2
Changed lines of the file:
@@
 F 0 "J2" H 8700 5150 50  0000 C CNN
 F 1 "Screw_Terminal_01x02" H 8700 4800 50  0000 C CNN
-F 2 "custom:TERMINAL_BLOCK_1x2" H 8700 5050 50  0001 C CNN
+F 2 "TerminalBlock:TerminalBlock_bornier-2_P5.08mm" H 8700 5050 50  0001 C CNN
 F 3 "~" H 8700 5050 50  0001 C CNN
 	1    8700 5050
@@
 AR Path="/5E826FFF/5E835E8A" Ref="Q4"  Part="1"
 F 0 "Q4" H 4650 6450 50  0000 L CNN
-F 1 "NP" H 4650 6550 50  0000 L CNN
+F 1 "NP_PNP_CBE" H 4650 6550 50  0000 L CNN
 F 2 "Package_TO_SOT_THT:TO-92" H 4650 6600 50  0001 C CNN
 F 3 "~" H 4450 6500 50  0001 C CNN
@@
 AR Path="/5E826FFF/5E835E91" Ref="Q3"  Part="1"
 F 0 "Q3" H 4650 5650 50  0000 L CNN
-F 1 "NP" H 4650 5550 50  0000 L CNN
+F 1 "NP_NPN_CBE" H 4650 5550 50  0000 L CNN
 F 2 "Package_TO_SOT_THT:TO-92" H 4650 5700 50  0001 C CNN
 F 3 "~" H 4450 5600 50  0001 C CNN
@@
 AR Path="/5E826FFF/5E857044" Ref="R23"  Part="1"
 F 0 "R23" V 4650 6850 50  0000 L CNN
-F 1 "NP_10k" V 4550 6860 31  0000 L CNN
+F 1 "NP_47" V 4550 6860 31  0000 L CNN
 F 2 "Resistor_THT:R_Axial_DIN0207_L6.3mm_D2.5mm_P10.16mm_Horizontal" V 4480 6950 50  0001 C CNN
 F 3 "~" H 4550 6950 50  0001 C CNN
@@
 AR Path="/5E826FFF/5E85714B" Ref="R19"  Part="1"
 F 0 "R19" V 4650 5050 50  0000 L CNN
-F 1 "NP_10k" V 4550 5060 31  0000 L CNN
+F 1 "NP_47" V 4550 5060 31  0000 L CNN
 F 2 "Resistor_THT:R_Axial_DIN0207_L6.3mm_D2.5mm_P10.16mm_Horizontal" V 4480 5150 50  0001 C CNN
 F 3 "~" H 4550 5150 50  0001 C CNN
@@
 AR Path="/5E826FFF/5E8668D9" Ref="R20"  Part="1"
 F 0 "R20" V 4100 5800 50  0000 L CNN
-F 1 "NP_10k" V 4000 5810 31  0000 L CNN
+F 1 "NP_3k3" V 4000 5810 31  0000 L CNN
 F 2 "Resistor_THT:R_Axial_DIN0207_L6.3mm_D2.5mm_P10.16mm_Horizontal" V 3930 5900 50  0001 C CNN
 F 3 "~" H 4000 5900 50  0001 C CNN
@@
 AR Path="/5E826FFF/5E87F9FD" Ref="JP6"  Part="1"
 F 0 "JP6" H 3150 5980 50  0000 C CNN
-F 1 "SolderJumper_2_Bridged" H 3150 5800 50  0001 C CNN
+F 1 "SolderJumper_Bridged" H 3150 5800 50  0001 C CNN
 F 2 "Jumper:SolderJumper-2_P1.3mm_Open_RoundedPad1.0x1.5mm" H 3150 5900 50  0001 C CNN
 F 3 "~" H 3150 5900 50  0001 C CNN
@@
 AR Path="/5E826FFF/5E7FBE4A" Ref="R25"  Part="1"
 F 0 "R25" V 4100 6400 50  0000 L CNN
-F 1 "NP_10k" V 4000 6410 31  0000 L CNN
+F 1 "NP_3k3" V 4000 6410 31  0000 L CNN
 F 2 "Resistor_THT:R_Axial_DIN0207_L6.3mm_D2.5mm_P10.16mm_Horizontal" V 3930 6500 50  0001 C CNN
 F 3 "~" H 4000 6500 50  0001 C CNN
@@
 AR Path="/5E826FFF/5E7FBEA6" Ref="R24"  Part="1"
 F 0 "R24" V 4100 5500 50  0000 L CNN
-F 1 "NP_10k" V 4000 5510 31  0000 L CNN
+F 1 "NP_3k3" V 4000 5510 31  0000 L CNN
 F 2 "Resistor_THT:R_Axial_DIN0207_L6.3mm_D2.5mm_P10.16mm_Horizontal" V 3930 5600 50  0001 C CNN
 F 3 "~" H 4000 5600 50  0001 C CNN
@@
 P 3000 1850
 AR Path="/5E4A013A/5EC0B44C" Ref="C?"  Part="1"
-AR Path="/5E826FFF/5EC0B44C" Ref="C?"  Part="1"
-F 0 "C?" H 3025 1950 50  0000 L CNN
+AR Path="/5E826FFF/5EC0B44C" Ref="C7"  Part="1"
+F 0 "C7" H 3025 1950 50  0000 L CNN
 F 1 "10nF" H 3025 1750 50  0000 L CNN
 F 2 "Capacitor_THT:C_Disc_D3.0mm_W1.6mm_P2.50mm" H 3038 1700 50  0001 C CNN
@@
 $EndComp
 $Comp
-L custom:PASSIVE_BUZZER BZ?
+L custom:PASSIVE_BUZZER BZ1
 U 1 1 5EC190CC
 P 3650 3800
-F 0 "BZ?" H 3800 3850 50  0000 L CNN
+F 0 "BZ1" H 3800 3850 50  0000 L CNN
 F 1 "PASSIVE_BUZZER" H 3800 3750 50  0001 L CNN
 F 2 "Buzzer_Beeper:Buzzer_TDK_PS1240P02BT_D12.2mm_H6.5mm" H 4225 3650 50  0001 C CNN

Commit message: automated commit
Parts:
- renumbered JP6 to JP3, R18 to R16, R19 to R17, R24 to R18, R25 to R19, R23 to R21, TP18 to TP12
Changed lines of the file:
@@
 	3000 1700 3000 1450
 $Comp
-L Device:R R18
+L Device:R R16
 U 1 1 5E8344F0
 P 7700 5050
-F 0 "R18" V 7600 5000 50  0000 C CNN
+F 0 "R16" V 7600 5000 50  0000 C CNN
 F 1 "80" V 7700 5050 50  0000 C CNN
 F 2 "Resistor_THT:R_Axial_DIN0207_L6.3mm_D2.5mm_P10.16mm_Horizontal" V 7630 5050 50  0001 C CNN
@@
 AR Path="/5E4A00FF/5E857044" Ref="R?"  Part="1"
 AR Path="/5E4A013A/5E857044" Ref="R?"  Part="1"
-AR Path="/5E826FFF/5E857044" Ref="R23"  Part="1"
-F 0 "R23" V 4650 6850 50  0000 L CNN
+AR Path="/5E826FFF/5E857044" Ref="R21"  Part="1"
+F 0 "R21" V 4650 6850 50  0000 L CNN
 F 1 "NP_47" V 4550 6860 31  0000 L CNN
 F 2 "Resistor_THT:R_Axial_DIN0207_L6.3mm_D2.5mm_P10.16mm_Horizontal" V 4480 6950 50  0001 C CNN
@@
 AR Path="/5E4A00FF/5E85714B" Ref="R?"  Part="1"
 AR Path="/5E4A013A/5E85714B" Ref="R?"  Part="1"
-AR Path="/5E826FFF/5E85714B" Ref="R19"  Part="1"
-F 0 "R19" V 4650 5050 50  0000 L CNN
+AR Path="/5E826FFF/5E85714B" Ref="R17"  Part="1"
+F 0 "R17" V 4650 5050 50  0000 L CNN
 F 1 "NP_47" V 4550 5060 31  0000 L CNN
 F 2 "Resistor_THT:R_Axial_DIN0207_L6.3mm_D2.5mm_P10.16mm_Horizontal" V 4480 5150 50  0001 C CNN
@@
 AR Path="/5E4A00FF/5E87F9FD" Ref="JP?"  Part="1"
 AR Path="/5E4A013A/5E87F9FD" Ref="JP?"  Part="1"
-AR Path="/5E826FFF/5E87F9FD" Ref="JP6"  Part="1"
-F 0 "JP6" H 3150 5980 50  0000 C CNN
+AR Path="/5E826FFF/5E87F9FD" Ref="JP3"  Part="1"
+F 0 "JP3" H 3150 5980 50  0000 C CNN
 F 1 "SolderJumper_Bridged" H 3150 5800 50  0001 C CNN
 F 2 "Jumper:SolderJumper-2_P1.3mm_Open_RoundedPad1.0x1.5mm" H 3150 5900 50  0001 C CNN
@@
 AR Path="/5E4A00FF/5E880781" Ref="TP?"  Part="1"
 AR Path="/5E4A013A/5E880781" Ref="TP?"  Part="1"
-AR Path="/5E826FFF/5E880781" Ref="TP18"  Part="1"
-F 0 "TP18" H 4900 6050 50  0000 L BNN
+AR Path="/5E826FFF/5E880781" Ref="TP12"  Part="1"
+F 0 "TP12" H 4900 6050 50  0000 L BNN
 F 1 "PTH_1_mm" H 4700 5950 50  0001 L BNN
 F 2 "custom:TestPoint_THTPad_D2.0mm_Drill1.0mm" H 4650 5800 50  0001 L BNN
@@
 AR Path="/5E4A00FF/5E7FBE4A" Ref="R?"  Part="1"
 AR Path="/5E4A013A/5E7FBE4A" Ref="R?"  Part="1"
-AR Path="/5E826FFF/5E7FBE4A" Ref="R25"  Part="1"
-F 0 "R25" V 4100 6400 50  0000 L CNN
+AR Path="/5E826FFF/5E7FBE4A" Ref="R19"  Part="1"
+F 0 "R19" V 4100 6400 50  0000 L CNN
 F 1 "NP_3k3" V 4000 6410 31  0000 L CNN
 F 2 "Resistor_THT:R_Axial_DIN0207_L6.3mm_D2.5mm_P10.16mm_Horizontal" V 3930 6500 50  0001 C CNN
@@
 AR Path="/5E4A00FF/5E7FBEA6" Ref="R?"  Part="1"
 AR Path="/5E4A013A/5E7FBEA6" Ref="R?"  Part="1"
-AR Path="/5E826FFF/5E7FBEA6" Ref="R24"  Part="1"
-F 0 "R24" V 4100 5500 50  0000 L CNN
+AR Path="/5E826FFF/5E7FBEA6" Ref="R18"  Part="1"
+F 0 "R18" V 4100 5500 50  0000 L CNN
 F 1 "NP_3k3" V 4000 5510 31  0000 L CNN
 F 2 "Resistor_THT:R_Axial_DIN0207_L6.3mm_D2.5mm_P10.16mm_Horizontal" V 3930 5600 50  0001 C CNN
