File: synth/POWER.sch (KiCad schematic (older format))
At the start: 9 parts

Commit message: automated commit
Parts:
- removed JP?: SolderJumper_2_Open, symbol Jumper:SolderJumper_2_Open
- added C4, C5: NP, symbol Device:CP1
- added D2: D_Schottky_Small_ALT, symbol Device:D_Schottky_Small_ALT
- added J1: 9V_BAT_HOLDER, symbol Connector_Generic:Conn_01x02
- added SW2: SW_SPDT, symbol Switch:SW_SPDT
- gave numbers to parts that had none: 8
Connections:
- net +5V: now also C5.1
- net GND: now also C4.2, C5.2, J1.2 (Pin_2)
- net VDD_BAT: now also C4.1, SW2.1 (A)
- new net: D2.2 (A), J1.1 (Pin_1)
- new net: D2.1 (K), SW2.2 (B)
- no-connect marks 0 -> 1
Other:
- note added: "+"
- note added: "-"
- note removed: "NEED TO ADD BATTERY HOLDER"
- note removed: "SILKSCREEN:\nWARNING: DO NOT CONNECT\nUNLESS BOARD IS CONVERTED\nTO OPERATE AT HIGHER VOLTAGES.\nALTERNATIVE PARTS REQUIRED."
- moved on the sheet: TP13, TP14, TP15

Commit message: automated commit
Other:
- moved on the sheet: C4, C5, C6, D2, J1, R14, R15, SW2, TP13, TP14, TP15, TP16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

Commit message: automated commit
Parts:
- C4, C5, C6: footprint (none) -> Capacitor_THT:CP_Radial_D6.3mm_P2.50mm
- D2: footprint (none) -> Diode_THT:D_DO-41_SOD81_P10.16mm_Horizontal
- J1: footprint (none) -> custom:BC9VPC
- R14, R15: footprint (none) -> Resistor_THT:R_Axial_DIN0207_L6.3mm_D2.5mm_P10.16mm_Horizontal
- SW2: footprint (none) -> custom:OS102011MS2QN1
- renumbered TP16 to TP13, TP13 to TP14, TP14 to TP16
Other:
- moved on the sheet: D2
Changed lines of the file:
@@
 F 0 "R15" V 6425 4450 50  0000 L CNN
 F 1 "10k" V 6350 4400 39  0000 L CNN
-F 2 "" V 6280 4450 50  0001 C CNN
+F 2 "Resistor_THT:R_Axial_DIN0207_L6.3mm_D2.5mm_P10.16mm_Horizontal" V 6280 4450 50  0001 C CNN
 F 3 "~" H 6350 4450 50  0001 C CNN
 	1    6350 4450
@@
 F 0 "R14" V 6425 3750 50  0000 L CNN
 F 1 "10k" V 6350 3700 39  0000 L CNN
-F 2 "" V 6280 3750 50  0001 C CNN
+F 2 "Resistor_THT:R_Axial_DIN0207_L6.3mm_D2.5mm_P10.16mm_Horizontal" V 6280 3750 50  0001 C CNN
 F 3 "~" H 6350 3750 50  0001 C CNN
 	1    6350 3750
@@
 AR Path="/5E69BCFF" Ref="#PWR?"  Part="1"
 AR Path="/5E4A00E6/5E69BCFF" Ref="#PWR?"  Part="1"
-AR Path="/5E69BAF5/5E69BCFF" Ref="#PWR024"  Part="1"
-F 0 "#PWR024" H 6350 4550 50  0001 C CNN
+AR Path="/5E69BAF5/5E69BCFF" Ref="#PWR025"  Part="1"
+F 0 "#PWR025" H 6350 4550 50  0001 C CNN
 F 1 "GND" H 6355 4627 50  0000 C CNN
 F 2 "" H 6350 4800 50  0001 C CNN
@@
 AR Path="/5E4A00E6/5E69BD18" Ref="#PWR?"  Part="1"
 AR Path="/5E69BD18" Ref="#PWR?"  Part="1"
-AR Path="/5E69BAF5/5E69BD18" Ref="#PWR017"  Part="1"
-F 0 "#PWR017" H 3550 3900 50  0001 C CNN
+AR Path="/5E69BAF5/5E69BD18" Ref="#PWR020"  Part="1"
+F 0 "#PWR020" H 3550 3900 50  0001 C CNN
 F 1 "VDD_BAT" H 3200 4000 50  0000 L BNN
 F 2 "" H 3350 3850 50  0001 C CNN
@@
 AR Path="/5E69BD28" Ref="#PWR?"  Part="1"
 AR Path="/5E4A00E6/5E69BD28" Ref="#PWR?"  Part="1"
-AR Path="/5E69BAF5/5E69BD28" Ref="#PWR019"  Part="1"
-F 0 "#PWR019" H 4200 4500 50  0001 C CNN
+AR Path="/5E69BAF5/5E69BD28" Ref="#PWR023"  Part="1"
+F 0 "#PWR023" H 4200 4500 50  0001 C CNN
 F 1 "GND" H 4205 4577 50  0000 C CNN
 F 2 "" H 4200 4750 50  0001 C CNN
@@
 AR Path="/5E4A00E6/5E69BD12" Ref="#PWR?"  Part="1"
 AR Path="/5E69BD12" Ref="#PWR?"  Part="1"
-AR Path="/5E69BAF5/5E69BD12" Ref="#PWR023"  Part="1"
-F 0 "#PWR023" H 6350 3350 50  0001 C CNN
+AR Path="/5E69BAF5/5E69BD12" Ref="#PWR019"  Part="1"
+F 0 "#PWR019" H 6350 3350 50  0001 C CNN
 F 1 "+5V" H 6350 3640 50  0000 C CNN
 F 2 "" H 6350 3500 50  0001 C CNN
@@
 P 6700 3900
 AR Path="/5E4A00E6/5E61F9DD" Ref="TP?"  Part="1"
-AR Path="/5E69BAF5/5E61F9DD" Ref="TP16"  Part="1"
-F 0 "TP16" V 6800 3850 50  0000 L BNN
+AR Path="/5E69BAF5/5E61F9DD" Ref="TP13"  Part="1"
+F 0 "TP13" V 6800 3850 50  0000 L BNN
 F 1 "PTH_1_mm" V 6850 3700 50  0001 L BNN
 F 2 "TestPoint:TestPoint_THTPad_D2.0mm_Drill1.0mm" H 6500 3650 50  0001 L BNN
@@
 P 3150 4050
 AR Path="/5E4A00E6/5E6200E9" Ref="TP?"  Part="1"
-AR Path="/5E69BAF5/5E6200E9" Ref="TP13"  Part="1"
-F 0 "TP13" H 3200 4050 50  0000 L BNN
+AR Path="/5E69BAF5/5E6200E9" Ref="TP14"  Part="1"
+F 0 "TP14" H 3200 4050 50  0000 L BNN
 F 1 "PTH_1_mm" V 3300 3850 50  0001 L BNN
 F 2 "TestPoint:TestPoint_THTPad_D2.0mm_Drill1.0mm" H 2950 3800 50  0001 L BNN
@@
 P 4400 4550
 AR Path="/5E4A00E6/5E62014F" Ref="TP?"  Part="1"
-AR Path="/5E69BAF5/5E62014F" Ref="TP14"  Part="1"
-F 0 "TP14" H 4450 4550 50  0000 L BNN
+AR Path="/5E69BAF5/5E62014F" Ref="TP16"  Part="1"
+F 0 "TP16" H 4450 4550 50  0000 L BNN
 F 1 "PTH_1_mm" V 4550 4350 50  0001 L BNN
 F 2 "TestPoint:TestPoint_THTPad_D2.0mm_Drill1.0mm" H 4200 4300 50  0001 L BNN
@@
 F 0 "C6" H 7125 4550 50  0000 L CNN
 F 1 "NP" H 7125 4350 50  0000 L CNN
-F 2 "" H 7100 4450 50  0001 C CNN
+F 2 "Capacitor_THT:CP_Radial_D6.3mm_P2.50mm" H 7100 4450 50  0001 C CNN
 F 3 "~" H 7100 4450 50  0001 C CNN
 	1    7100 4450
@@
 F 0 "C5" H 4825 4500 50  0000 L CNN
 F 1 "NP" H 4825 4300 50  0000 L CNN
-F 2 "" H 4800 4400 50  0001 C CNN
+F 2 "Capacitor_THT:CP_Radial_D6.3mm_P2.50mm" H 4800 4400 50  0001 C CNN
 F 3 "~" H 4800 4400 50  0001 C CNN
 	1    4800 4400
@@
 AR Path="/5E77E00E" Ref="#PWR?"  Part="1"
 AR Path="/5E4A00E6/5E77E00E" Ref="#PWR?"  Part="1"
-AR Path="/5E69BAF5/5E77E00E" Ref="#PWR020"  Part="1"
-F 0 "#PWR020" H 4800 4500 50  0001 C CNN
+AR Path="/5E69BAF5/5E77E00E" Ref="#PWR024"  Part="1"
+F 0 "#PWR024" H 4800 4500 50  0001 C CNN
 F 1 "GND" H 4805 4577 50  0000 C CNN
 F 2 "" H 4800 4750 50  0001 C CNN
@@
 F 0 "C4" H 3675 4500 50  0000 L CNN
 F 1 "NP" H 3675 4300 50  0000 L CNN
-F 2 "" H 3650 4400 50  0001 C CNN
+F 2 "Capacitor_THT:CP_Radial_D6.3mm_P2.50mm" H 3650 4400 50  0001 C CNN
 F 3 "~" H 3650 4400 50  0001 C CNN
 	1    3650 4400
@@
 AR Path="/5E77E1EF" Ref="#PWR?"  Part="1"
 AR Path="/5E4A00E6/5E77E1EF" Ref="#PWR?"  Part="1"
-AR Path="/5E69BAF5/5E77E1EF" Ref="#PWR018"  Part="1"
-F 0 "#PWR018" H 3650 4500 50  0001 C CNN
+AR Path="/5E69BAF5/5E77E1EF" Ref="#PWR022"  Part="1"
+F 0 "#PWR022" H 3650 4500 50  0001 C CNN
 F 1 "GND" H 3655 4577 50  0000 C CNN
 F 2 "" H 3650 4750 50  0001 C CNN
@@
 F 0 "J1" H 5250 2200 50  0000 C CNN
 F 1 "9V_BAT_HOLDER" H 5250 1800 50  0000 C CNN
-F 2 "" H 5250 2100 50  0001 C CNN
+F 2 "custom:BC9VPC" H 5250 2100 50  0001 C CNN
 F 3 "~" H 5250 2100 50  0001 C CNN
 	1    5250 2100
@@
 AR Path="/5E4A00E6/5E781AC9" Ref="#PWR?"  Part="1"
 AR Path="/5E781AC9" Ref="#PWR?"  Part="1"
-AR Path="/5E69BAF5/5E781AC9" Ref="#PWR025"  Part="1"
-F 0 "#PWR025" H 7000 1850 50  0001 C CNN
+AR Path="/5E69BAF5/5E781AC9" Ref="#PWR017"  Part="1"
+F 0 "#PWR017" H 7000 1850 50  0001 C CNN
 F 1 "VDD_BAT" H 6650 1950 50  0000 L BNN
 F 2 "" H 6800 1800 50  0001 C CNN
@@
 AR Path="/5E7825BB" Ref="#PWR?"  Part="1"
 AR Path="/5E4A00E6/5E7825BB" Ref="#PWR?"  Part="1"
-AR Path="/5E69BAF5/5E7825BB" Ref="#PWR022"  Part="1"
-F 0 "#PWR022" H 5950 2200 50  0001 C CNN
+AR Path="/5E69BAF5/5E7825BB" Ref="#PWR018"  Part="1"
+F 0 "#PWR018" H 5950 2200 50  0001 C CNN
 F 1 "GND" H 5955 2277 50  0000 C CNN
 F 2 "" H 5950 2450 50  0001 C CNN
@@
 L Device:D_Schottky_Small_ALT D?
 U 1 1 5E7840DC
-P 5700 2100
+P 5750 2100
 AR Path="/5E4A00FF/5E7840DC" Ref="D?"  Part="1"
 AR Path="/5E4A013A/5E7840DC" Ref="D?"  Part="1"
 AR Path="/5E69BAF5/5E7840DC" Ref="D2"  Part="1"
-F 0 "D2" H 5800 2050 50  0000 L CNN
-F 1 "D_Schottky_Small_ALT" H 5420 2020 50  0001 L CNN
-F 2 "" V 5700 2100 50  0001 C CNN
-F 3 "~" V 5700 2100 50  0001 C CNN
-F 4 "" H 5550 2050 50  0000 C CNN "NP"
-	1    5700 2100
+F 0 "D2" H 5850 2050 50  0000 L CNN
+F 1 "D_Schottky_Small_ALT" H 5470 2020 50  0001 L CNN
+F 2 "Diode_THT:D_DO-41_SOD81_P10.16mm_Horizontal" V 5750 2100 50  0001 C CNN
+F 3 "~" V 5750 2100 50  0001 C CNN
+F 4 "" H 5600 2050 50  0000 C CNN "NP"
+	1    5750 2100
 	-1   0    0    1
 $EndComp
 Wire Wire Line
-	5450 2100 5600 2100
+	5450 2100 5650 2100
 Connection ~ 3650 4050
 Text Notes 5050 2150 0    63   ~ 0
@@
 F 0 "SW2" H 6250 2270 50  0000 C CNN
 F 1 "SW_SPDT" H 6250 1900 50  0001 C CNN
-F 2 "" H 6250 2100 50  0001 C CNN
+F 2 "custom:OS102011MS2QN1" H 6250 2100 50  0001 C CNN
 F 3 "" H 6250 2100 50  0001 C CNN
 	1    6250 2100
@@
 $EndComp
 Wire Wire Line
-	5800 2100 6050 2100
+	5850 2100 6050 2100
 Wire Wire Line
 	6450 2000 6800 2000

Commit message: automated commit
Parts:
- TP13, TP14, TP15, TP16: footprint TestPoint:TestPoint_THTPad_D2.0mm_Drill1.0mm -> custom:TestPoint_THTPad_D2.0mm_Drill1.0mm
Changed lines of the file:
@@
 F 0 "TP13" V 6800 3850 50  0000 L BNN
 F 1 "PTH_1_mm" V 6850 3700 50  0001 L BNN
-F 2 "TestPoint:TestPoint_THTPad_D2.0mm_Drill1.0mm" H 6500 3650 50  0001 L BNN
+F 2 "custom:TestPoint_THTPad_D2.0mm_Drill1.0mm" H 6500 3650 50  0001 L BNN
 F 3 "" H 6700 4000 50  0001 L BNN
 	1    6700 3900
@@
 F 0 "TP15" H 5300 4050 50  0000 L BNN
 F 1 "PTH_1_mm" V 5400 3850 50  0001 L BNN
-F 2 "TestPoint:TestPoint_THTPad_D2.0mm_Drill1.0mm" H 5050 3800 50  0001 L BNN
+F 2 "custom:TestPoint_THTPad_D2.0mm_Drill1.0mm" H 5050 3800 50  0001 L BNN
 F 3 "" H 5250 4150 50  0001 L BNN
 	1    5250 4050
@@
 F 0 "TP14" H 3200 4050 50  0000 L BNN
 F 1 "PTH_1_mm" V 3300 3850 50  0001 L BNN
-F 2 "TestPoint:TestPoint_THTPad_D2.0mm_Drill1.0mm" H 2950 3800 50  0001 L BNN
+F 2 "custom:TestPoint_THTPad_D2.0mm_Drill1.0mm" H 2950 3800 50  0001 L BNN
 F 3 "" H 3150 4150 50  0001 L BNN
 	1    3150 4050
@@
 F 0 "TP16" H 4450 4550 50  0000 L BNN
 F 1 "PTH_1_mm" V 4550 4350 50  0001 L BNN
-F 2 "TestPoint:TestPoint_THTPad_D2.0mm_Drill1.0mm" H 4200 4300 50  0001 L BNN
+F 2 "custom:TestPoint_THTPad_D2.0mm_Drill1.0mm" H 4200 4300 50  0001 L BNN
 F 3 "" H 4400 4650 50  0001 L BNN
 	1    4400 4550
