File: synth/POWER.sch (KiCad schematic (older format))
At the start: 12 parts, among them J1 9V_BAT_HOLDER, SW2 SW_SPDT, U3 SCD7805BTG

Commit message: automated commit
Parts:
- removed D2: D_Schottky_Small_ALT, Diode_THT:D_DO-41_SOD81_P10.16mm_Horizontal, symbol Device:D_Schottky_Small_ALT
- added D2: Diode, Diode_THT:D_DO-41_SOD81_P10.16mm_Horizontal, symbol Device:D_Small_ALT
- gave numbers to parts that had none: 2
Connections:
- net at J1.1 (Pin_1): now also D2.2 (A)
- net at SW2.2 (B): now also D2.1 (K)
Changed lines of the file:
@@
 	1    0    0    -1
-$EndComp
-$Comp
-L Device:D_Schottky_Small_ALT D?
-U 1 1 5E7840DC
-P 5750 2100
-AR Path="/5E4A00FF/5E7840DC" Ref="D?"  Part="1"
-AR Path="/5E4A013A/5E7840DC" Ref="D?"  Part="1"
-AR Path="/5E69BAF5/5E7840DC" Ref="D2"  Part="1"
-F 0 "D2" H 5850 2050 50  0000 L CNN
-F 1 "D_Schottky_Small_ALT" H 5470 2020 50  0001 L CNN
-F 2 "Diode_THT:D_DO-41_SOD81_P10.16mm_Horizontal" V 5750 2100 50  0001 C CNN
-F 3 "~" V 5750 2100 50  0001 C CNN
-F 4 "" H 5600 2050 50  0000 C CNN "NP"
-	1    5750 2100
-	-1   0    0    1
 $EndComp
 Wire Wire Line
@@
 AR Path="/5E4A013A/5EC0A5D4" Ref="C?"  Part="1"
 AR Path="/5E826FFF/5EC0A5D4" Ref="C?"  Part="1"
-AR Path="/5E69BAF5/5EC0A5D4" Ref="C?"  Part="1"
-F 0 "C?" H 7125 4550 50  0000 L CNN
+AR Path="/5E69BAF5/5EC0A5D4" Ref="C6"  Part="1"
+F 0 "C6" H 7125 4550 50  0000 L CNN
 F 1 "10nF" H 7125 4350 50  0000 L CNN
 F 2 "Capacitor_THT:C_Disc_D3.0mm_W1.6mm_P2.50mm" H 7138 4300 50  0001 C CNN
@@
 AR Path="/5E4A013A/5EC0DC78" Ref="C?"  Part="1"
 AR Path="/5E826FFF/5EC0DC78" Ref="C?"  Part="1"
-AR Path="/5E69BAF5/5EC0DC78" Ref="C?"  Part="1"
-F 0 "C?" H 4825 4500 50  0000 L CNN
+AR Path="/5E69BAF5/5EC0DC78" Ref="C5"  Part="1"
+F 0 "C5" H 4825 4500 50  0000 L CNN
 F 1 "10nF" H 4825 4300 50  0000 L CNN
 F 2 "Capacitor_THT:C_Disc_D3.0mm_W1.6mm_P2.50mm" H 4838 4250 50  0001 C CNN
@@
 Wire Wire Line
 	3650 4050 3850 4050
+$Comp
+L Device:D_Small_ALT D2
+U 1 1 5E8AADC5
+P 5750 2100
+F 0 "D2" H 5700 2180 50  0000 L CNN
+F 1 "Diode" H 5600 2020 50  0001 L CNN
+F 2 "Diode_THT:D_DO-41_SOD81_P10.16mm_Horizontal" V 5750 2100 50  0001 C CNN
+F 3 "~" V 5750 2100 50  0001 C CNN
+	1    5750 2100
+	-1   0    0    -1
+$EndComp
 $EndSCHEMATC
