File: synth/synth.kicad_pcb (KiCad board)
At the start: 2 copper layers, 75 parts, among them J1 9V_BAT_HOLDER, J2 Screw_Terminal_01x02, Q1 Q_NMOS_SGD, Q2 Q_PMOS_SGD, Q3 Q_NPN_CBE, Q4 Q_PNP_CBE, SW1 SW_SPDT, SW2 SW_SPDT, SW3 SW_SPDT, U1 MCP6004, U2 SE555P, U3 SCD7805BTG, U4 MCP6002

Commit message: automated commit
Parts:
- added G***: LOGO, custom:rivet_logo, F.Cu at (134.5, 91.7)
- added R24: NP_10k, Resistor_THT:R_Axial_DIN0207_L6.3mm_D2.5mm_P10.16mm_Horizontal, F.Cu at (183.9, 136.6)
- added R25: NP_10k, Resistor_THT:R_Axial_DIN0207_L6.3mm_D2.5mm_P10.16mm_Horizontal, F.Cu at (178.1, 142.6)
- TP1, TP10, TP11, TP12, TP13, TP17, TP18, TP2, TP3, TP4, TP5, TP6, TP7, TP8, TP9: footprint TestPoint:TestPoint_THTPad_D2.0mm_Drill1.0mm -> custom:TestPoint_THTPad_D2.0mm_Drill1.0mm
- TP14, TP15, TP16: footprint TestPoint:TestPoint_THTPad_D2.0mm_Drill1.0mm -> custom:TestPoint_THTPad_D2.0mm_Drill1.0mm; moved to B.Cu
- U4: footprint Package_DIP:DIP-8_W7.62mm -> Package_DIP:DIP-8_W7.62mm_Socket
- moved JP1 472.2 mm to (133.4, 63.0), turned to 45 degrees
- moved R3 460.8 mm to (133.5, 56.2), turned to 225 degrees
- moved U1 396.5 mm to (117.5, 102.7), turned to 315 degrees
- moved C3 395.5 mm to (109.5, 102.7), turned to 135 degrees
- moved RV2 389.9 mm to (140.2, 43.5), turned to 135 degrees
- moved C2 388.5 mm to (103.5, 110.7), turned to 45 degrees
- moved Q2 369.1 mm to (122.7, 82.2), turned to 270 degrees
- moved Q1 363.5 mm to (105.0, 82.2), turned to 270 degrees
- moved RV1 356.2 mm to (78.0, 88.6), turned to 315 degrees
- moved U4 353.2 mm to (168.3, 131.2), turned to 315 degrees
- moved C7 350.1 mm to (178.0, 131.4), turned to 135 degrees
- moved JP2 336.6 mm to (118.4, 57.8), turned to 135 degrees
- moved R10 332.3 mm to (110.2, 58.2), turned to 315 degrees
- moved D1 326.8 mm to (108.1, 66.0), turned to 315 degrees
- moved R11 321.7 mm to (100.3, 68.1), turned to 315 degrees
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Connections:
- Q3 pad 2: Net-(JP6-Pad1) -> Net-(Q3-Pad2)
- Q4 pad 2: Net-(JP6-Pad1) -> Net-(Q4-Pad2)
Routing:
- net /MAIN_VFO/TRIANGLE: track 0.00 -> 43.8 mm
- net Net-(JP6-Pad2): track 0.00 -> 36.2 mm
- net /MAIN_VFO/DISCHARGE: track 0.00 -> 35.6 mm
- net Net-(R8-Pad2): track 0.00 -> 33.9 mm
- net Net-(JP5-Pad1): track 0.00 -> 26.8 mm
- net Net-(Q1-Pad3): track 0.00 -> 20.6 mm
- net Net-(R5-Pad1): track 0.00 -> 17.3 mm
- net /OUTPUT/LO_Z_REF: track 0.00 -> 17.0 mm
- net Net-(R8-Pad1): track 0.00 -> 16.6 mm
- net Net-(C2-Pad2): track 0.00 -> 13.8 mm
- net Net-(JP4-Pad2): track 0.00 -> 13.5 mm
- net Net-(JP4-Pad1): track 0.00 -> 9.95 mm
- net Net-(JP7-Pad1): track 0.00 -> 8.61 mm
- net /OUTPUT/OUTPUT: track 0.00 -> 8.16 mm
- net Net-(JP6-Pad1): track 0.00 -> 8.11 mm
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- added copper zone on F.Cu, net +5V
- added copper zone on B.Cu, net GND
Other:
- board outline added: 153.6 x 153.9 mm
- board text added: "OFF"
- board text added: "ON"
- board text added: "POWER"
- board text added: "SPEAKER"
