File: synth/synth.kicad_pcb (KiCad board)
At the start: 2 copper layers, 153.6 x 153.9 mm, 69 parts, among them J1 9V_BAT_HOLDER, J2 Screw_Terminal_01x02, Q1 Q_NMOS_SGD, Q2 Q_PMOS_SGD, Q3 NP_NPN_CBE, Q4 NP_PNP_CBE, SW1 SW_SPDT, SW2 SW_SPDT, SW3 SW_SPDT, U1 MCP6004, U2 SE555P, U3 SCD7805BTG, U4 MCP6002

Commit message: automated commit
Parts:
- J2: footprint TerminalBlock:TerminalBlock_bornier-2_P5.08mm -> custom:TerminalBlock_D2_P5.08mm
- moved RV5 133.3 mm to (99.9, 96.2), turned to 225 degrees
- moved BZ1 47.8 mm to (162.9, 95.4)
- moved TP10 32.9 mm to (116.7, 121.6)
- moved R10 21.6 mm to (96.3, 82.4), turned to 315 degrees
- moved C7 3.64 mm to (176.2, 134.1), turned to 135 degrees
- moved R8 2.70 mm to (120.3, 126.2)
- moved J2 2.51 mm to (162.6, 162.6)
- turned JP2 to 225 degrees
- turned JP3 to 225 degrees
Routing:
- net /MAIN_VFO/TRIM: track 0.00 -> 59.1 mm, vias 0 -> 2
- net Net-(JP2-Pad1): track 4.95 -> 61.0 mm, vias 0 -> 2
- net Net-(JP6-Pad2): track 93.5 -> 56.3 mm
- net Net-(JP4-Pad1): track 30.1 -> 0.00 mm, vias 1 -> 0
- net HI_Z_REF: track 134.9 -> 161.1 mm, vias 2 -> 3
- net Net-(JP4-Pad2): track 26.1 -> 0.00 mm
- net /OUTPUT/LO_Z_REF: track 105.9 -> 82.2 mm, vias 3 -> 2
- net Net-(SW1-Pad3): track 0.00 -> 16.4 mm
- net VDD_BAT: track 47.6 -> 33.5 mm
- net +5V: track 48.9 -> 60.9 mm, vias 5 -> 0
- net Net-(JP5-Pad1): track 9.79 -> 0.00 mm
- net Net-(JP7-Pad1): track 8.61 -> 0.00 mm
- net GND: track 72.3 -> 79.2 mm, vias 0 -> 2
- net Net-(R10-Pad2): track 0.00 -> 5.49 mm
- net Net-(R12-Pad1): track 0.00 -> 5.22 mm
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
Commit message: automated commit
Parts:
- added JP4: SolderJumper_Open, Jumper:SolderJumper-2_P1.3mm_Open_RoundedPad1.0x1.5mm, F.Cu at (38.3, 24.1)
- added JP5: SolderJumper_Open, Jumper:SolderJumper-2_P1.3mm_Open_RoundedPad1.0x1.5mm, F.Cu at (34.0, 38.7)
- added JP7: SolderJumper_Open, Jumper:SolderJumper-2_P1.3mm_Open_RoundedPad1.0x1.5mm, F.Cu at (63.2, -4.90)
- added R13: 1k, Resistor_THT:R_Axial_DIN0207_L6.3mm_D2.5mm_P10.16mm_Horizontal, F.Cu at (33.1, 19.6)
- added R16: 1k, Resistor_THT:R_Axial_DIN0207_L6.3mm_D2.5mm_P10.16mm_Horizontal, F.Cu at (29.1, 33.9)
- added R17: 1k, Resistor_THT:R_Axial_DIN0207_L6.3mm_D2.5mm_P10.16mm_Horizontal, F.Cu at (57.9, -0.22)
- J2: footprint custom:TerminalBlock_D2_P5.08mm -> TerminalBlock:TerminalBlock_bornier-2_P5.08mm
- Q2: footprint Package_TO_SOT_THT:TO-92 -> custom:TO-92_one_off
Connections:
- Q1 pad 1: Net-(Q1-Pad1) -> Net-(JP5-Pad1)
- Q2 pad 1: Net-(Q2-Pad1) -> Net-(JP7-Pad2)
- R1 pad 2: Net-(R1-Pad2) -> Net-(JP4-Pad2)
- RV1 pad 1: (no net) -> Net-(RV1-Pad1)
- RV1 pad 3: Net-(R1-Pad2) -> Net-(JP4-Pad1)
- RV2 pad 1: Net-(Q1-Pad1) -> Net-(JP5-Pad2)
- RV2 pad 3: Net-(Q2-Pad1) -> Net-(JP7-Pad1)
- RV3 pad 1: (no net) -> Net-(RV3-Pad1)
- SW2 pad 3: (no net) -> Net-(SW2-Pad3)
- SW3 pad 3: (no net) -> Net-(SW3-Pad3)
- U1 pad 2: Net-(R1-Pad2) -> Net-(JP4-Pad2)
- U2 pad 5: (no net) -> Net-(U2-Pad5)
Other:
- board text added: "1k0"

Commit message: automated commit
Parts:
- removed JP4, JP5, JP7: SolderJumper_Open, Jumper:SolderJumper-2_P1.3mm_Open_RoundedPad1.0x1.5mm
- removed JP6: SolderJumper_Bridged, Jumper:SolderJumper-2_P1.3mm_Open_RoundedPad1.0x1.5mm
- removed R23: NP_47, Resistor_THT:R_Axial_DIN0207_L6.3mm_D2.5mm_P10.16mm_Horizontal
- removed R24, R25: NP_3k3, Resistor_THT:R_Axial_DIN0207_L6.3mm_D2.5mm_P10.16mm_Horizontal
- removed TP18: PTH_1_mm, custom:TestPoint_THTPad_D2.0mm_Drill1.0mm
- added R21: NP_47, Resistor_THT:R_Axial_DIN0207_L6.3mm_D2.5mm_P10.16mm_Horizontal, F.Cu at (178.9, 149.1)
- added TP12: PTH_1_mm, custom:TestPoint_THTPad_D2.0mm_Drill1.0mm, F.Cu at (200.3, 135.9)
- C2: value 10nF -> 100nF
- JP1, JP2: value SolderJumper_Bridged -> SolderJumper_Open
- JP3: value SolderJumper_Open -> SolderJumper_Bridged
- Q1: value Q_NMOS_SGD -> 2N3904; footprint Package_TO_SOT_THT:TO-92 -> Package_TO_SOT_THT:TO-92_Inline
- Q2: value Q_PMOS_SGD -> 2N3906; footprint custom:TO-92_one_off -> Package_TO_SOT_THT:TO-92_Inline
- R10, R11, R12, R13, RV5: value 1k -> 1k0
- R16: value 1k -> 80
- R17: value 1k -> NP_47
- R18: value 80 -> NP_3k3
- R19: value NP_47 -> NP_3k3
- R3: value NP_100 -> 1k0
- moved R17 200.8 mm to (197.3, 144.3), turned to 135 degrees
- moved R16 185.6 mm to (168.3, 156.6), turned to 90 degrees
- moved JP3 102.0 mm to (163.1, 145.1), turned to 315 degrees
- moved R13 98.1 mm to (88.5, 100.5), turned to 270 degrees
- moved JP2 34.9 mm to (84.3, 105.2), turned to 270 degrees
- moved R18 25.4 mm to (183.9, 136.6), turned to 315 degrees
- moved R19 19.6 mm to (177.9, 142.4), turned to 315 degrees
- moved R3 10.2 mm to (127.9, 61.5), turned to 45 degrees
- moved R12 3.10 mm to (95.0, 100.3), turned to 270 degrees
- moved Q1 2.63 mm to (105.2, 84.8), turned to 90 degrees
- moved Q2 2.55 mm to (122.3, 87.5), turned to 90 degrees
Connections:
- JP2 pad 2: /MAIN_VFO/TRIM -> Net-(JP2-Pad2)
- JP3 pad 1: HI_Z_REF -> Net-(JP3-Pad1)
- JP3 pad 2: Net-(JP2-Pad1) -> Net-(JP3-Pad2)
- Q1 pad 1: Net-(JP5-Pad1) -> Net-(Q1-Pad1)
- Q2 pad 1: Net-(JP7-Pad2) -> Net-(Q1-Pad1)
- Q2 pad 3: Net-(Q1-Pad3) -> Net-(Q2-Pad3)
- Q3 pad 3: Net-(JP6-Pad2) -> Net-(JP3-Pad2)
- Q4 pad 3: Net-(JP6-Pad2) -> Net-(JP3-Pad2)
- R1 pad 2: Net-(JP4-Pad2) -> Net-(JP2-Pad2)
- R13 pad 1: Net-(JP4-Pad1) -> Net-(JP2-Pad1)
- R13 pad 2: Net-(JP4-Pad2) -> Net-(JP2-Pad2)
- R16 pad 1: Net-(JP5-Pad1) -> /OUTPUT/OUTPUT
- R16 pad 2: Net-(JP5-Pad2) -> VFO_OUT
- R17 pad 1: Net-(JP7-Pad1) -> +5V
- R17 pad 2: Net-(JP7-Pad2) -> Net-(Q3-Pad1)
- R18 pad 1: /OUTPUT/OUTPUT -> Net-(Q3-Pad2)
- R18 pad 2: VFO_OUT -> Net-(JP3-Pad1)
- R19 pad 1: +5V -> Net-(Q4-Pad2)
- R19 pad 2: Net-(Q3-Pad1) -> Net-(JP3-Pad1)
- R20 pad 1: Net-(JP6-Pad2) -> Net-(JP3-Pad2)
- R20 pad 2: Net-(JP6-Pad1) -> Net-(JP3-Pad1)
- R3 pad 1: Net-(JP1-Pad2) -> Net-(C2-Pad2)
- R3 pad 2: Net-(C2-Pad2) -> Net-(JP1-Pad2)
- RV1 pad 1: Net-(RV1-Pad1) -> (no net)
- RV1 pad 2: Net-(Q1-Pad3) -> Net-(Q1-Pad1)
- RV1 pad 3: Net-(JP4-Pad1) -> Net-(JP2-Pad1)
- RV2 pad 1: Net-(JP5-Pad2) -> Net-(Q1-Pad3)
- RV2 pad 3: Net-(JP7-Pad1) -> Net-(Q2-Pad3)
- RV3 pad 1: Net-(RV3-Pad1) -> (no net)
- SW2 pad 3: Net-(SW2-Pad3) -> (no net)
- SW3 pad 3: Net-(SW3-Pad3) -> (no net)
- TP3 pad 1: Net-(Q1-Pad3) -> Net-(Q1-Pad1)
- U1 pad 1: Net-(Q1-Pad3) -> Net-(Q1-Pad1)
- U1 pad 2: Net-(JP4-Pad2) -> Net-(JP2-Pad2)
- U1 pad 5: Net-(JP2-Pad1) -> /MAIN_VFO/TRIM
- U2 pad 5: Net-(U2-Pad5) -> (no net)
- U4 pad 6: Net-(JP6-Pad2) -> Net-(JP3-Pad2)
- U4 pad 7: Net-(JP6-Pad1) -> Net-(JP3-Pad1)
Routing:
- net HI_Z_REF: track 161.1 -> 51.2 mm, vias 3 -> 0
- net Net-(R1-Pad2): track 78.3 -> 0.00 mm, vias 1 -> 0
- net Net-(JP6-Pad2): track 56.3 -> 0.00 mm
- net Net-(JP3-Pad2): track 0.00 -> 56.3 mm
- net Net-(JP2-Pad2): track 0.00 -> 53.5 mm, vias 0 -> 1
- net Net-(Q2-Pad3): track 0.00 -> 45.7 mm, vias 0 -> 1
- net Net-(Q2-Pad1): track 45.7 -> 0.00 mm, vias 1 -> 0
- net Net-(JP6-Pad1): track 42.4 -> 0.00 mm
- net Net-(JP3-Pad1): track 0.00 -> 42.4 mm
- net Net-(JP2-Pad1): track 61.0 -> 33.6 mm, vias 2 -> 0
- net Net-(Q1-Pad3): track 66.6 -> 58.7 mm, vias 0 -> 1
- net Net-(Q1-Pad1): track 58.7 -> 66.6 mm, vias 1 -> 0
- net /MAIN_VFO/TRIM: track 59.1 -> 64.7 mm
- net GND: track 79.2 -> 76.9 mm
- net Net-(Q2-Pad2): track 7.92 -> 6.71 mm
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
Commit message: automated commit
Other:
- board text added: "https://github.com/DJ027X/simple_synth/ REV 3.0"
- board text removed: "https://github.com/DJ027X/simple_synth/"
